File: PCB/ultrasonic.kicad_sch (KiCad schematic)
At the start: 27 parts, among them J1 HC-SR04, J2 USB C, J3 SG92R, U1 STM32F103C8Tx, U2 CH340N

Commit message: PCB: ready, 3.3v will be from blue pill connection to powerbank ToDo: WPF scale from 4m to 2m max range, step case
Parts:
- added C13, C14: 33pF, symbol Device:C
- added C15: 220µF, symbol Device:C_Polarized
- added D4: LED, symbol Device:LED
- added J4: SWD, symbol Connector:Conn_01x04_Pin
- added R6: 1K, Resistor_SMD:R_0805_2012Metric, symbol Device:R_US
- added R7: 10k, Resistor_SMD:R_0805_2012Metric, symbol Device:R_US
- added Y1: 8MHz, symbol Device:Crystal
- C12: value 10uF -> 100nF
Connections:
- net +3.3V: now also J4.1 (Pin_1), R6.1; no longer C5.1, C6.1, FB1.1, J1.1 (Pin_1), U1.9 (VDDA)
- net +5V: now also C2.1, C3.1, F1.2, J1.1 (Pin_1), J3.2 (Pin_2), U2.5 (VCC), C15.1; no longer F1.1, J2.A4 (VBUS), J2.A9 (VBUS), J2.B4 (VBUS), J2.B9 (VBUS), J3.1 (Pin_1)
- net at U1.2 (PC13): now also D4.1 (K)
- net SWDIO: now reaches U1.34 (PA13)
- net SWDIO: now also J4.2 (Pin_2)
- net SWCLK: now reaches U1.37 (PA14)
- net SWCLK: now also J4.3 (Pin_3)
- net at U1.44 (BOOT0): now also R7.2
- net HSE_IN: now reaches U1.5 (PD0)
- net HSE_IN: now also C13.1, Y1.2
- net HSE_OUT: now reaches U1.6 (PD1)
- net HSE_OUT: now also C14.2, Y1.1
- new net: F1.1, J2.A4 (VBUS), J2.A9 (VBUS), J2.B4 (VBUS), J2.B9 (VBUS)
- new net: C13.2, C14.1
- new net: C15.2, J3.1 (Pin_1)
- new net: D4.2 (A), R6.2
- new net +3.3VA: C5.1, C6.1, FB1.1, U1.9 (VDDA)
- no-connect marks 0 -> 1
Other:
- moved on the sheet: C1, C10, C11, C12, C2, C3, C4, C5, C6, C7, C8, C9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

Commit message: sch fix CAD work started
Parts:
- removed F1: Fuse, symbol Device:Fuse
- added C16, C17: 1µF, symbol Device:C
- added J4: Powerbank, symbol Connector:Conn_01x02_Pin
- added U2: XC6206P332MR, Package_TO_SOT_SMD:SOT-23-3, symbol Regulator_Linear:XC6206PxxxMR
Connections:
- net +3.3V: now also C16.2, U2.2 (VO)
- net +5V: now also C17.2, J4.1 (Pin_1), U2.3 (VI); no longer C2.1, C3.1, R5.2, U2.5 (VCC)
- net at J2.A4 (VBUS), J2.A9 (VBUS), J2.B4 (VBUS)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: now also C2.1, C3.1, R5.2, U2.5 (VCC)
- new net: C16.1, C17.1, U2.1 (GND)
Other:
- moved on the sheet: C10, C11, C12, C13, C14, C15, C2, C3, C4, C5, C6, C7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

Commit message: Tests on prototype, clean up code
Parts:
- renumbered J4 to J5, U2 to U3
Changed lines of the file:
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@@
 		(in_pos_files yes)
 		(dnp no)
-		(property "Reference" "U2"
+		(property "Reference" "U3"
 			(at 379.73 177.8 0)
 			(show_name no)
@@
 			(project "ultrasonic"
 				(path "/289eb5d8-08cd-4918-afaa-21b9428315d9"
-					(reference "U2")
+					(reference "U3")
 					(unit 1)
 				)
@@
 		(in_pos_files yes)
 		(dnp no)
-		(property "Reference" "J4"
+		(property "Reference" "J5"
 			(at 313.69 95.25 0)
 			(show_name no)
@@
 			(project "ultrasonic"
 				(path "/289eb5d8-08cd-4918-afaa-21b9428315d9"
-					(reference "J4")
+					(reference "J5")
 					(unit 1)
 				)
